File: Hardware/KiCad/CANTranslate/CANTranslate.kicad_sch (KiCad schematic)
At the start: 43 parts, among them J1 USB_C_Receptacle_USB2.0_16P, J2 Conn_01x05_Pin, J3 SM04B-GHS-TB(LF)(SN), J4 SM04B-GHS-TB(LF)(SN), SW1 SW_Push, SW2 SW_SPDT, SW3 SW_SPST, U1 USBLC6-2SC6, U2 STM32F103C8T6, U3 AMS1117-3.3, U4 TPS2116DRL, U5 SN65HVD230, Y1 16MHz

Commit message: git shenanigans
Parts:
- removed J3: SM04B-GHS-TB(LF)(SN), Connector_JST:JST_GH_SM04B-GHS-TB_1x04-1MP_P1.25mm_Horizontal, symbol CustomParts:SM04B-GHS-CAN-HEADER
- removed R1: 1k5, Resistor_SMD:R_0402_1005Metric, symbol Device:R
- removed R2: 10k, Resistor_SMD:R_0402_1005Metric, symbol Device:R
- removed U2: STM32F103C8T6, Package_QFP:LQFP-48_7x7mm_P0.5mm, symbol MCU_ST_STM32F1:STM32F103C8Tx
- added C12, C13: 2u2, Capacitor_SMD:C_0402_1005Metric, symbol Device:C
- added C2: 100n, Capacitor_SMD:C_0402_1005Metric, symbol Device:C
- added J4: SM04B-GHS-TB(LF)(SN), Connector_JST:JST_GH_SM04B-GHS-TB_1x04-1MP_P1.25mm_Horizontal, symbol CustomParts:SM04B-GHS-CAN-HEADER
- added R10: 120, Resistor_SMD:R_0402_1005Metric, symbol Device:R
- added R4: 470, Resistor_SMD:R_0402_1005Metric, symbol Device:R
- added SW4: SW_SPST, DSIC01LSGET:SW-SMD_DSIC01LSGET, symbol Switch:SW_SPST
- added U2: STM32F205RGT6, Package_QFP:LQFP-64_10x10mm_P0.5mm, symbol MCU_ST_STM32F2:STM32F205RGTx
- added U6: SN65HVD230, Package_SO:SOIC-8_3.9x4.9mm_P1.27mm, symbol Interface_CAN_LIN:SN65HVD230
- SW2: footprint Button_Switch_THT:SW_Slide_SPDT_Straight_CK_OS102011MS2Q -> easyeda2kicad:SW-TH_SS12D07VG4; LCSC C221829 -> C2939726
- renumbered C9 to C10, C10 to C11, C11 to C14, C12 to C15, C2 to C3, C3 to C4, C4 to C5, C5 to C6, C6 to C7, C7 to C8, C8 to C9, J4 to J3, R3 to R1, R4 to R2, R5 to R3, R6 to R5, R7 to R6, R8 to R7, R9 to R8, R10 to R9
Connections:
- net +3.3V: now also C2.1, U2.1 (VBAT), U2.13 (VDDA), U2.19 (VDD), U2.32 (VDD), U2.48 (VDD), U2.64 (VDD), U6.3 (VCC)
- net +5V: now also J4.1; no longer J3.1
- net BOOT0: now also U2.60 (BOOT0)
- net GND: now also C12.2, C13.2, C2.2, J4.4, U2.12 (VSSA), U2.18 (VSS), U2.63 (VSS), U6.2 (GND), U6.8 (Rs)
- net HSE_IN: now also U2.5 (PH0)
- net HSE_OUT: now also R4.1, U2.6 (PH1); no longer C11.1
- net NRST: now also U2.7 (NRST)
- net SWCLK: now also U2.49 (PA14)
- net SWDIO: now also U2.46 (PA13)
- net SWO: now also U2.55 (PB3)
- net USB_D+: now also U2.45 (PA12)
- net USB_D-: now also U2.44 (PA11)
- net CAN+ renamed CAN1+
- net CAN- renamed CAN1-
- net CAN_RX renamed CAN1_RX
- net CAN1_RX: now also U2.61 (PB8)
- net CAN_TX renamed CAN1_TX
- net CAN1_TX: now also U2.62 (PB9)
- new net: C11.1, R4.2
- new net: R10.2, SW4.2 (B)
- new net CAN2+: J4.2, R10.1, U6.7 (CANH)
- new net CAN2-: J4.3, SW4.1 (A), U6.6 (CANL)
- new net CAN2_RX: U2.33 (PB12), U6.4 (R)
- new net CAN2_TX: U2.34 (PB13), U6.1 (D)
- new net VCAP_1: C12.1, U2.31 (VCAP_1)
- new net VCAP_2: C13.1, U2.47 (VCAP_2)
- no-connect marks 31 -> 45
Other:
- note added: "CAN TRANSCEIVERS AND CONNECTORS"
- note added: "MOUNTING HOLES AND FIDUCIALS"
- note removed: "CAN TRANSCEIVER AND CONNECTORS"
- note removed: "STM32 MCU"
- moved on the sheet: C1, C3, C4, C5, C6, C7, C8, C9, FID1, FID2, FID3, H1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
